File: magloop_pico.kicad_pcb (KiCad board)
At the start: 2 copper layers, 99.6 x 99.9 mm, 102 parts, among them J1 Conn_Coaxial_Power, J10 5V AUDIO MUTE, J2 Conn_02x03_Odd_Even, J3 POWER SW, J4 Conn_02x03_Odd_Even, J5 Conn_02x04_Odd_Even, J6 TO RF RELAY, J7 ETHERNET, J8 5-1634513-1, J9 12V AUDIO MUTE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

Commit message: Added BOMs from Digikey and Kicad schematic.  Minor clean up top metal and changed 50 ohm resistors to 51.
Parts:
- R13, R14, R15, R16: value 50.0 -> 51.0
Connections:
- J2 pad 1: /AUTOTUNE -> /EXIT
- J2 pad 3: /EXIT -> /AUTOTUNE
- U4 pad 10: /EXIT -> /AUTOTUNE
- U4 pad 11: /AUTOTUNE -> /EXIT
Routing:
- net /EXIT: track 107.3 -> 101.0 mm
- net /AUTOTUNE: track 101.0 -> 107.3 mm
- net GND: vias 158 -> 160
